File: openevse-ac-filter.brd (EAGLE design)
At the start: 64.9 x 23.5 mm, 7 parts

Commit message: bump v2.1
Parts:
- removed F1: (no value), fuse:GSH15
- added F2: (no value), fuse-20mm:GSH15
Connections:
- net N$2: now also F2.2; no longer F1.2
- net N$5: now also F2.1; no longer F1.1
Routing:
- net N$19: track 0.00 -> 38.2 mm
- net N$2: track 30.8 -> 12.5 mm
- net N$16: track 0.00 -> 7.84 mm
- net N$18: track 0.00 -> 7.69 mm
- net N$20: track 0.00 -> 6.61 mm
- net N$15: track 0.00 -> 3.88 mm
Other:
- board size 64.9 x 23.5 mm -> 64.9 x 23.9 mm
- board text added: "OpenEVSE AC Filter V2.1"
- board text removed: "OpenEVSE AC Filter V2.0"
Changed lines of the file:
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@@
 <setting verticaltext="up"/>
 </settings>
-<grid distance="0.5" unitdist="mm" unit="mm" style="lines" multiple="1" display="yes" altdistance="0.025" altunitdist="inch" altunit="inch"/>
+<grid distance="0.2" unitdist="mm" unit="mm" style="lines" multiple="1" display="yes" altdistance="0.025" altunitdist="inch" altunit="inch"/>
 <layers>
-<layer number="1" name="Top" color="4" fill="1" visible="yes" active="yes"/>
+<layer number="1" name="Top" color="4" fill="1" visible="no" active="yes"/>
 <layer number="16" name="Bottom" color="1" fill="1" visible="yes" active="yes"/>
 <layer number="17" name="Pads" color="2" fill="1" visible="yes" active="yes"/>
@@
 <board>
 <plain>
-<wire x1="2.532" y1="0" x2="67.468" y2="0" width="0" layer="20"/>
-<wire x1="67.468" y1="0" x2="67.468" y2="23.5" width="0" layer="20"/>
+<wire x1="2.532" y1="-0.4" x2="67.468" y2="-0.4" width="0" layer="20"/>
+<wire x1="67.468" y1="-0.4" x2="67.468" y2="23.5" width="0" layer="20"/>
 <wire x1="67.468" y1="23.5" x2="2.532" y2="23.5" width="0" layer="20"/>
-<wire x1="2.532" y1="23.5" x2="2.532" y2="0" width="0" layer="20"/>
+<wire x1="2.532" y1="23.5" x2="2.532" y2="-0.4" width="0" layer="20"/>
 <text x="26" y="19.5" size="1.016" layer="25" font="vector" ratio="18">U2 RN214</text>
 <hole x="11.5" y="11.5" drill="3.2"/>
@@
 <text x="4.524" y="-0.984" size="1.27" layer="21" font="vector" ratio="18">OpenEVSE
 AC Filter
-V2.0
+V2.1
 </text>
 <text x="14" y="12" size="1.27" layer="21" font="vector" ratio="18">L1
 </text>
-<text x="57.5" y="1" size="1.27" layer="21" font="vector" ratio="18">L1
+<text x="57.7" y="1" size="1.27" layer="21" font="vector" ratio="18">L1
 BROWN</text>
 <text x="4" y="13.5" size="1.27" layer="21" font="vector" ratio="18">N</text>
@@
 <element name="U$2" library="Schaffner-CM-Choke" package="RN214-0.3-02-47M" value="RN214-0.3-02-47M" x="37.57" y="23.34" smashed="yes" rot="R180"/>
 <element name="C1" library="capacitor-wima" package="C5B2.5" value="10F" x="42.7" y="11.44" smashed="yes" rot="R90">
-<attribute name="NAME" x="45.092" y="16.676" size="1.27" layer="25" font="vector" ratio="18" rot="R180"/>
+<attribute name="NAME" x="46.892" y="14.276" size="1.27" layer="25" font="vector" ratio="18" rot="R180"/>
 </element>
 <element name="C2" library="capacitor-wima" package="C5B2.5" value="10nF" x="17.5" y="11" smashed="yes" rot="R90">
@@
 <attribute name="MF" value="" x="49.652" y="3.628" size="1.778" layer="27" display="off"/>
 <attribute name="MPN" value="237-103" x="49.652" y="3.628" size="1.778" layer="27" display="off"/>
-<attribute name="NAME" x="45.9982" y="5.5638" size="1.27" layer="25" ratio="10"/>
+<attribute name="NAME" x="46.1982" y="5.5638" size="1.27" layer="25" ratio="10"/>
 <attribute name="OC_FARNELL" value="unknown" x="49.652" y="3.628" size="1.778" layer="27" display="off"/>
 <attribute name="OC_NEWARK" value="18M7116" x="49.652" y="3.628" size="1.778" layer="27" display="off"/>
@@
 <attribute name="VALUE" x="15.2608" y="24.2956" size="1.27" layer="27" ratio="10" rot="R180"/>
 </element>
-<element name="F1" library="fuse" library_urn="urn:adsk.eagle:library:233" package="GSH15" package3d_urn="urn:adsk.eagle:package:14065/1" value="" x="57.4" y="19.8" smashed="yes" rot="R180">
-<attribute name="MF" value="" x="57.4" y="19.8" size="1.778" layer="27" rot="R180" display="off"/>
-<attribute name="MPN" value="64900001039" x="57.4" y="19.8" size="1.778" layer="27" rot="R180" display="off"/>
-<attribute name="NAME" x="58.1804" y="16.1932" size="1.778" layer="25" ratio="10" rot="R180"/>
-<attribute name="OC_FARNELL" value="1271673" x="57.4" y="19.8" size="1.778" layer="27" rot="R180" display="off"/>
-<attribute name="OC_NEWARK" value="02P0318" x="57.4" y="19.8" size="1.778" layer="27" rot="R180" display="off"/>
-<attribute name="POPULARITY" value="3" x="57.4" y="19.8" size="1.778" layer="27" rot="R180" display="off"/>
-<attribute name="VALUE" x="61.8196" y="25.261" size="1.778" layer="27" ratio="10" rot="R180"/>
+<element name="F2" library="fuse-20mm" package="GSH15" package3d_urn="urn:adsk.eagle:package:14065/1" value="" x="57.5" y="19.8" smashed="yes" rot="R180">
+<attribute name="MF" value="" x="57.5" y="19.8" size="1.778" layer="27" rot="R180" display="off"/>
+<attribute name="MPN" value="64900001039" x="57.5" y="19.8" size="1.778" layer="27" rot="R180" display="off"/>
+<attribute name="NAME" x="58.4196" y="16.1932" size="1.778" layer="25" ratio="10" rot="R180"/>
+<attribute name="OC_FARNELL" value="1271673" x="57.5" y="19.8" size="1.778" layer="27" rot="R180" display="off"/>
+<attribute name="OC_NEWARK" value="02P0318" x="57.5" y="19.8" size="1.778" layer="27" rot="R180" display="off"/>
+<attribute name="POPULARITY" value="3" x="57.5" y="19.8" size="1.778" layer="27" rot="R180" display="off"/>
+<attribute name="VALUE" x="58.4196" y="25.261" size="1.778" layer="27" ratio="10" rot="R180"/>
 </element>
 </elements>
@@
 <wire x1="36.07" y1="16.84" x2="39.95" y2="16.84" width="2.032" layer="1"/>
 <wire x1="39.95" y1="16.84" x2="40.18" y2="17.07" width="2.032" layer="1"/>
-<wire x1="40.894" y1="17.784" x2="40.18" y2="17.07" width="2.032" layer="1"/>
+<wire x1="40.18" y1="17.07" x2="40.894" y2="17.784" width="2.032" layer="1"/>
 <wire x1="40.18" y1="17.07" x2="40.18" y2="16.5" width="2.032" layer="1"/>
 <wire x1="40.18" y1="16.5" x2="42.7" y2="13.98" width="2.032" layer="1"/>
-<contactref element="F1" pad="2"/>
-<wire x1="40.18" y1="17.07" x2="42.91" y2="19.8" width="2.032" layer="1"/>
-<wire x1="42.91" y1="19.8" x2="49.78" y2="19.8" width="2.032" layer="1"/>
-<wire x1="40.18" y1="17.07" x2="42.91" y2="19.8" width="2.032" layer="16"/>
-<wire x1="42.91" y1="19.8" x2="49.78" y2="19.8" width="2.032" layer="16"/>
+<contactref element="F2" pad="2"/>
+<wire x1="40.894" y1="17.784" x2="41.4" y2="18.29" width="2.02" layer="1"/>
+<wire x1="41.4" y1="18.29" x2="41.4" y2="18.4" width="2.02" layer="1"/>
+<wire x1="41.4" y1="18.4" x2="42.8" y2="19.8" width="2.02" layer="1"/>
+<wire x1="42.8" y1="19.8" x2="43.12" y2="19.8" width="2.02" layer="1"/>
 </signal>
 <signal name="N$3">
@@
 <signal name="N$5">
 <contactref element="X1" pad="3"/>
-<contactref element="F1" pad="1"/>
 <wire x1="54.652" y1="2.338" x2="65.02" y2="12.706" width="2.032" layer="1"/>
-<wire x1="65.02" y1="12.706" x2="65.02" y2="19.8" width="2.032" layer="1"/>
+<contactref element="F2" pad="1"/>
+<wire x1="65.02" y1="12.706" x2="65.12" y2="12.806" width="2.02" layer="1"/>
+<wire x1="65.12" y1="12.806" x2="65.12" y2="19.8" width="2.02" layer="1"/>
 </signal>
 <signal name="N$7">
 <wire x1="54.5" y1="2.5" x2="65" y2="13" width="2.032" layer="16"/>
-<wire x1="65" y1="13" x2="65" y2="20" width="2.032" layer="16"/>
+<wire x1="65.2" y1="19.8" x2="65.2" y2="13.2" width="2.02" layer="16"/>
+<wire x1="65.2" y1="13.2" x2="65" y2="13" width="2.02" layer="16"/>
+</signal>
+<signal name="N$15">
+<wire x1="40.2" y1="17.2" x2="42.8" y2="19.8" width="2.02" layer="16"/>
+<wire x1="42.8" y1="19.8" x2="43" y2="19.8" width="2.02" layer="16"/>
+</signal>
+<signal name="N$16">
+<wire x1="36" y1="6.8" x2="38.2" y2="6.8" width="2.02" layer="1"/>
+<wire x1="38.2" y1="6.8" x2="38.6" y2="6.4" width="2.02" layer="1"/>
+<wire x1="38.6" y1="6.4" x2="41.2" y2="9" width="2.02" layer="1"/>
+<wire x1="41.2" y1="9" x2="42.6" y2="9" width="2.02" layer="1"/>
+</signal>
+<signal name="N$18">
+<wire x1="44.8" y1="2.4" x2="42.4" y2="2.4" width="2.02" layer="1"/>
+<wire x1="40.2" y1="4.6" x2="40.2" y2="4.8" width="2.02" layer="1"/>
+<wire x1="40.2" y1="4.8" x2="38.8" y2="6.2" width="2.02" layer="1"/>
+<wire x1="42.4" y1="2.4" x2="40.2" y2="4.6" width="2.02" layer="1"/>
+</signal>
+<signal name="N$19">
+<wire x1="24" y1="6.8" x2="20.6" y2="6.8" width="2.02" layer="16"/>
+<wire x1="20.6" y1="6.8" x2="20.6" y2="5.2" width="2.02" layer="16"/>
+<wire x1="20.6" y1="5.2" x2="18" y2="2.6" width="2.02" layer="16"/>
+<wire x1="18" y1="2.6" x2="8.2" y2="2.6" width="2.02" layer="16"/>
+<wire x1="8.2" y1="2.6" x2="4.8" y2="6" width="2.02" layer="16"/>
+<wire x1="4.8" y1="6" x2="4.8" y2="20.6" width="2.02" layer="16"/>
+<wire x1="4.8" y1="20.6" x2="5" y2="20.8" width="2.02" layer="16"/>
+</signal>
+<signal name="N$20">
+<wire x1="15" y1="20.6" x2="18.4" y2="17.2" width="2.02" layer="16"/>
+<wire x1="18.4" y1="17.2" x2="20.2" y2="17.2" width="2.02" layer="16"/>
 </signal>
 </signals>

Commit message: v2.2
Parts:
- removed C1: 10F, capacitor-wima:C5B2.5
- removed C2: 10nF, capacitor-wima:C5B2.5
- added C3, C4: DE2F3KY103MA3BM02F, DE2F3KY103MA3BM02F:DE2F3KY103MA3BM02F
- moved X1 10.8 mm to (60.5, 3.83)
- moved F2 4.40 mm to (61.9, 20.0)
- moved X2 1.02 mm to (8.96, 19.5)
Connections:
- removed net N$1: C1.1, U$1.P$4, U$2.P$4, X1.1
- removed net N$2: C1.2, F2.2, U$1.P$2, U$2.P$2
- removed net N$4: C2.2, U$1.P$1, U$2.P$1, X2.1
- new net N$17: C4.2, U$1.P$4, U$2.P$4, X1.1
- new net N$21: C3.1, U$1.P$1, U$2.P$1, X2.1
- new net N$22: C4.1, F2.2, U$1.P$2, U$2.P$2
- net N$3: now also C3.2; no longer C2.1
Routing:
- net N$17: track 0.00 -> 38.4 mm
- net N$19: track 38.2 -> 0.00 mm
- net N$21: track 0.00 -> 28.5 mm
- net N$22: track 0.00 -> 26.4 mm
- net N$1: track 22.3 -> 0.00 mm
- net N$7: track 21.7 -> 0.00 mm
- net N$4: track 16.4 -> 0.00 mm
- net N$2: track 12.5 -> 0.00 mm
- net N$16: track 7.84 -> 0.00 mm
- net N$18: track 7.69 -> 0.00 mm
- net N$20: track 6.61 -> 0.00 mm
- net N$11: track 5.69 -> 0.00 mm
- net N$12: track 5.54 -> 0.00 mm
- net N$13: track 4.42 -> 0.00 mm
- net N$10: track 4.35 -> 0.00 mm
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Other:
- board size 64.9 x 23.9 mm -> 73.5 x 23.9 mm
- board text added: "L1 B R O W N"
- board text added: "N B L U E"
- board text added: "OpenEVSE AC Filter V2.2"
- board text removed: "L1"
- board text removed: "N"
- board text removed: "NC"
- board text removed: "OpenEVSE AC Filter V2.1"
