File: openevse-ac-filter.sch (EAGLE design)
At the start: 7 parts

Commit message: bump v2.1
Parts:
- removed F1: (no value), fuse:GSH15
- added F2: (no value), fuse-20mm:GSH15
Connections:
- net N$2: now also F2.2; no longer F1.2
- net N$5: now also F2.1; no longer F1.1
Changed lines of the file:
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@@
 <part name="X1" library="con-wago-500" library_urn="urn:adsk.eagle:library:195" deviceset="W237-103" device="" package3d_urn="urn:adsk.eagle:package:10691/1"/>
 <part name="X2" library="con-wago-500" library_urn="urn:adsk.eagle:library:195" deviceset="W237-103" device="" package3d_urn="urn:adsk.eagle:package:10691/1"/>
-<part name="F1" library="fuse" library_urn="urn:adsk.eagle:library:233" deviceset="GSH15" device="" package3d_urn="urn:adsk.eagle:package:14065/1"/>
+<part name="F2" library="fuse-20mm" deviceset="GSH15" device="" package3d_urn="urn:adsk.eagle:package:14065/1"/>
 </parts>
 <sheets>
@@
 <attribute name="NAME" x="81.28" y="75.311" size="1.778" layer="95"/>
 </instance>
-<instance part="F1" gate="1" x="2.54" y="68.58" smashed="yes">
+<instance part="F2" gate="1" x="2.54" y="68.58" smashed="yes">
 <attribute name="NAME" x="-1.27" y="69.977" size="1.778" layer="95"/>
 <attribute name="VALUE" x="-1.27" y="65.659" size="1.778" layer="96"/>
@@
 <pinref part="U$2" gate="G$1" pin="P$2"/>
 <pinref part="C1" gate="G$1" pin="2"/>
-<wire x1="7.62" y1="68.58" x2="17.78" y2="68.58" width="0.1524" layer="91"/>
-<pinref part="F1" gate="1" pin="2"/>
-<junction x="7.62" y="68.58"/>
+<wire x1="10.16" y1="68.58" x2="17.78" y2="68.58" width="0.1524" layer="91"/>
 <wire x1="7.62" y1="68.58" x2="10.16" y2="68.58" width="0.1524" layer="91"/>
+<pinref part="F2" gate="1" pin="2"/>
 </segment>
 </net>
@@
 <segment>
 <pinref part="X1" gate="-3" pin="KL"/>
-<pinref part="F1" gate="1" pin="1"/>
 <wire x1="-2.54" y1="68.58" x2="-7.62" y2="68.58" width="0.1524" layer="91"/>
+<pinref part="F2" gate="1" pin="1"/>
 </segment>
 </net>

Commit message: v2.2
Parts:
- removed C1: 10F, capacitor-wima:C5/2.5
- removed C2: 10nF, capacitor-wima:C5/2.5
- added C3, C4: DE2F3KY103MA3BM02F, DE2F3KY103MA3BM02F:DE2F3KY103MA3BM02F
Connections:
- removed net N$1: C1.1, U$1.P$4, U$2.P$4, X1-1.KL
- removed net N$2: C1.2, F2.2, U$1.P$2, U$2.P$2
- removed net N$4: C2.2, U$1.P$1, U$2.P$1, X2-1.KL
- new net N$17: C4.2, U$1.P$4, U$2.P$4, X1-1.KL
- new net N$21: C3.1, U$1.P$1, U$2.P$1, X2-1.KL
- new net N$22: C4.1, F2.2, U$1.P$2, U$2.P$2
- net N$3: now also C3.2; no longer C2.1
Changed lines of the file:
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@@
 <?xml version="1.0" encoding="utf-8"?>
 <!DOCTYPE eagle SYSTEM "eagle.dtd">
-<eagle version="9.5.2">
+<eagle version="9.6.2">
 <drawing>
 <settings>
@@
 <part name="U$1" library="Schaffner-CM-Choke" deviceset="RN114-0.3-02-47M" device="" value="47mH"/>
 <part name="U$2" library="Schaffner-CM-Choke" deviceset="RN214-0.3-02-47M" device=""/>
-<part name="C1" library="capacitor-wima" deviceset="C" device="5/2.5" value="10F"/>
-<part name="C2" library="capacitor-wima" deviceset="C" device="5/2.5" value="10nF"/>
 <part name="X1" library="con-wago-500" library_urn="urn:adsk.eagle:library:195" deviceset="W237-103" device="" package3d_urn="urn:adsk.eagle:package:10691/1"/>
 <part name="X2" library="con-wago-500" library_urn="urn:adsk.eagle:library:195" deviceset="W237-103" device="" package3d_urn="urn:adsk.eagle:package:10691/1"/>
 <part name="F2" library="fuse-20mm" deviceset="GSH15" device="" package3d_urn="urn:adsk.eagle:package:14065/1"/>
+<part name="C3" library="DE2F3KY103MA3BM02F" deviceset="DE2F3KY103MA3BM02F" device=""/>
+<part name="C4" library="DE2F3KY103MA3BM02F" deviceset="DE2F3KY103MA3BM02F" device=""/>
 </parts>
 <sheets>
@@
 <instance part="U$1" gate="G$1" x="22.86" y="63.5" smashed="yes"/>
 <instance part="U$2" gate="G$1" x="22.86" y="63.5" smashed="yes"/>
-<instance part="C1" gate="G$1" x="10.16" y="73.66" smashed="yes">
-<attribute name="NAME" x="11.684" y="74.041" size="1.778" layer="95"/>
-<attribute name="VALUE" x="11.684" y="68.961" size="1.778" layer="96"/>
-</instance>
-<instance part="C2" gate="G$1" x="55.88" y="73.66" smashed="yes">
-<attribute name="NAME" x="57.404" y="74.041" size="1.778" layer="95"/>
-<attribute name="VALUE" x="57.404" y="68.961" size="1.778" layer="96"/>
-</instance>
 <instance part="X1" gate="-1" x="-12.7" y="78.74" smashed="yes">
 <attribute name="NAME" x="-12.7" y="79.629" size="1.778" layer="95" rot="R180"/>
@@
 <attribute name="VALUE" x="-1.27" y="65.659" size="1.778" layer="96"/>
 </instance>
+<instance part="C3" gate="G$1" x="60.96" y="68.58" smashed="yes" rot="R90">
+<attribute name="NAME" x="54.61" y="77.47" size="1.778" layer="95" rot="R90" align="center-left"/>
+<attribute name="VALUE" x="57.15" y="77.47" size="1.778" layer="96" rot="R90" align="center-left"/>
+</instance>
+<instance part="C4" gate="G$1" x="7.62" y="68.58" smashed="yes" rot="R90">
+<attribute name="NAME" x="1.27" y="77.47" size="1.778" layer="95" rot="R90" align="center-left"/>
+<attribute name="VALUE" x="3.81" y="77.47" size="1.778" layer="96" rot="R90" align="center-left"/>
+</instance>
 </instances>
 <busses>
 </busses>
 <nets>
-<net name="N$1" class="0">
-<segment>
-<pinref part="U$1" gate="G$1" pin="P$4"/>
-<pinref part="U$2" gate="G$1" pin="P$4"/>
-<pinref part="C1" gate="G$1" pin="1"/>
-<wire x1="17.78" y1="76.2" x2="10.16" y2="76.2" width="0.1524" layer="91"/>
-<wire x1="10.16" y1="76.2" x2="2.54" y2="76.2" width="0.1524" layer="91"/>
-<wire x1="2.54" y1="76.2" x2="2.54" y2="78.74" width="0.1524" layer="91"/>
-<pinref part="X1" gate="-1" pin="KL"/>
-<wire x1="2.54" y1="78.74" x2="-7.62" y2="78.74" width="0.1524" layer="91"/>
-</segment>
-</net>
-<net name="N$2" class="0">
-<segment>
-<pinref part="U$1" gate="G$1" pin="P$2"/>
-<pinref part="U$2" gate="G$1" pin="P$2"/>
-<pinref part="C1" gate="G$1" pin="2"/>
-<wire x1="10.16" y1="68.58" x2="17.78" y2="68.58" width="0.1524" layer="91"/>
-<wire x1="7.62" y1="68.58" x2="10.16" y2="68.58" width="0.1524" layer="91"/>
-<pinref part="F2" gate="1" pin="2"/>
-</segment>
-</net>
 <net name="N$3" class="0">
 <segment>
 <pinref part="U$1" gate="G$1" pin="P$3"/>
 <pinref part="U$2" gate="G$1" pin="P$3"/>
-<pinref part="C2" gate="G$1" pin="1"/>
-<wire x1="50.8" y1="76.2" x2="55.88" y2="76.2" width="0.1524" layer="91"/>
+<pinref part="C3" gate="G$1" pin="2"/>
+<wire x1="50.8" y1="76.2" x2="50.8" y2="81.28" width="0.1524" layer="91"/>
+<wire x1="50.8" y1="81.28" x2="60.96" y2="81.28" width="0.1524" layer="91"/>
+<wire x1="60.96" y1="81.28" x2="73.66" y2="81.28" width="0.1524" layer="91"/>
+<wire x1="73.66" y1="81.28" x2="73.66" y2="76.2" width="0.1524" layer="91"/>
 <pinref part="X2" gate="-3" pin="KL"/>
-<wire x1="55.88" y1="76.2" x2="76.2" y2="76.2" width="0.1524" layer="91"/>
-</segment>
-</net>
-<net name="N$4" class="0">
-<segment>
-<pinref part="U$1" gate="G$1" pin="P$1"/>
-<pinref part="U$2" gate="G$1" pin="P$1"/>
-<pinref part="C2" gate="G$1" pin="2"/>
-<wire x1="50.8" y1="68.58" x2="55.88" y2="68.58" width="0.1524" layer="91"/>
-<wire x1="66.04" y1="68.58" x2="55.88" y2="68.58" width="0.1524" layer="91"/>
-<pinref part="X2" gate="-1" pin="KL"/>
-<wire x1="76.2" y1="66.04" x2="66.04" y2="66.04" width="0.1524" layer="91"/>
-<wire x1="66.04" y1="66.04" x2="66.04" y2="68.58" width="0.1524" layer="91"/>
+<wire x1="73.66" y1="76.2" x2="76.2" y2="76.2" width="0.1524" layer="91"/>
 </segment>
 </net>
@@
 </segment>
 </net>
+<net name="N$17" class="0">
+<segment>
+<pinref part="U$1" gate="G$1" pin="P$4"/>
+<pinref part="U$2" gate="G$1" pin="P$4"/>
+<wire x1="17.78" y1="76.2" x2="17.78" y2="81.28" width="0.1524" layer="91"/>
+<pinref part="C4" gate="G$1" pin="2"/>
+<wire x1="17.78" y1="81.28" x2="7.62" y2="81.28" width="0.1524" layer="91"/>
+<wire x1="7.62" y1="81.28" x2="2.54" y2="81.28" width="0.1524" layer="91"/>
+<pinref part="X1" gate="-1" pin="KL"/>
+<wire x1="2.54" y1="78.74" x2="-7.62" y2="78.74" width="0.1524" layer="91"/>
+<wire x1="2.54" y1="81.28" x2="2.54" y2="78.74" width="0.1524" layer="91"/>
+</segment>
+</net>
+<net name="N$21" class="0">
+<segment>
+<pinref part="U$1" gate="G$1" pin="P$1"/>
+<pinref part="U$2" gate="G$1" pin="P$1"/>
+<pinref part="C3" gate="G$1" pin="1"/>
+<wire x1="50.8" y1="68.58" x2="60.96" y2="68.58" width="0.1524" layer="91"/>
+<pinref part="X2" gate="-1" pin="KL"/>
+<wire x1="76.2" y1="66.04" x2="60.96" y2="66.04" width="0.1524" layer="91"/>
+<wire x1="60.96" y1="68.58" x2="60.96" y2="66.04" width="0.1524" layer="91"/>
+</segment>
+</net>
+<net name="N$22" class="0">
+<segment>
+<pinref part="F2" gate="1" pin="2"/>
+<pinref part="C4" gate="G$1" pin="1"/>
+<pinref part="U$1" gate="G$1" pin="P$2"/>
+<pinref part="U$2" gate="G$1" pin="P$2"/>
+<wire x1="7.62" y1="68.58" x2="17.78" y2="68.58" width="0.1524" layer="91"/>
+</segment>
+</net>
